File: PCB/ATtinyRemote.brd (EAGLE design)
At the start: 49.5 x 27.3 mm, 14 parts, among them IC1 ATTINY85DIP8, Q1 BC547, Q2 16MHz, U1 IR_Emitter, U2 IR_Receiver, X1 USB-A-H

Commit message: Version 1.0 of the PCB
Gerber files for http://www.dorkbotpdx.org/wiki/pcb_order
Parts:
- added C3: 100nF, rcl:C025-025X050
- moved R2 1.37 mm to (30.5, 6.60)
Connections:
- net +5V: now also C3.1
- net GND: now also C3.2
Routing:
- net GND: track 5.61 -> 20.7 mm
- net +5V: track 51.2 -> 53.7 mm
- net N$7: track 3.33 -> 4.81 mm
- net N$8: track 4.34 -> 3.30 mm
Other:
- board size 49.5 x 27.3 mm -> 49.5 x 27.2 mm
