File: PCB/ATtinyRemote.sch (EAGLE design)
At the start: 14 parts, among them IC1 ATTINY85DIP8, Q1 BC547, Q2 16MHz, U1 IR_Emitter, U2 IR_Receiver, X1 USB-A-H

Commit message: Minor adjustments to make it work better in practice
Parts:
- renumbered LED1 to STATUS, S1 to RESET
Changed lines of the file:
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@@
 <part name="GND3" library="supply1" deviceset="GND" device=""/>
 <part name="P+1" library="supply1" deviceset="+5V" device=""/>
-<part name="S1" library="SparkFun" deviceset="TAC_SWITCH" device="PTH" value="RESET"/>
+<part name="RESET" library="SparkFun" deviceset="TAC_SWITCH" device="PTH" value="RESET"/>
 <part name="R1" library="resistor" deviceset="R-EU_" device="0207/10" value="10k"/>
 <part name="P+2" library="supply1" deviceset="+5V" device=""/>
@@
 <part name="P+4" library="supply1" deviceset="+5V" device=""/>
 <part name="GND6" library="supply1" deviceset="GND" device=""/>
-<part name="LED1" library="led" deviceset="LED" device="3MM"/>
+<part name="STATUS" library="led" deviceset="LED" device="3MM"/>
 <part name="GND7" library="supply1" deviceset="GND" device=""/>
 <part name="Q2" library="crystal" deviceset="CRYSTAL" device="HC49S" value="16MHz"/>
@@
 <instance part="GND3" gate="1" x="83.82" y="30.48"/>
 <instance part="P+1" gate="1" x="27.94" y="68.58"/>
-<instance part="S1" gate="S" x="63.5" y="35.56"/>
+<instance part="RESET" gate="S" x="63.5" y="35.56"/>
 <instance part="R1" gate="G$1" x="50.8" y="33.02" rot="R180"/>
 <instance part="P+2" gate="1" x="45.72" y="38.1"/>
@@
 <instance part="P+4" gate="1" x="10.16" y="68.58"/>
 <instance part="GND6" gate="1" x="10.16" y="45.72"/>
-<instance part="LED1" gate="G$1" x="58.42" y="78.74" rot="R180"/>
+<instance part="STATUS" gate="G$1" x="58.42" y="78.74" rot="R180"/>
 <instance part="GND7" gate="1" x="48.26" y="78.74"/>
 <instance part="Q2" gate="G$1" x="83.82" y="50.8" smashed="yes">
@@
 </segment>
 <segment>
-<pinref part="S1" gate="S" pin="3"/>
-<pinref part="S1" gate="S" pin="4"/>
+<pinref part="RESET" gate="S" pin="3"/>
+<pinref part="RESET" gate="S" pin="4"/>
 <wire x1="68.58" y1="35.56" x2="68.58" y2="33.02" width="0.1524" layer="91"/>
 <pinref part="GND4" gate="1" pin="GND"/>
@@
 </segment>
 <segment>
-<pinref part="LED1" gate="G$1" pin="C"/>
+<pinref part="STATUS" gate="G$1" pin="C"/>
 <wire x1="58.42" y1="83.82" x2="58.42" y2="86.36" width="0.1524" layer="91"/>
 <pinref part="GND7" gate="1" pin="GND"/>
@@
 <net name="N$3" class="0">
 <segment>
-<pinref part="S1" gate="S" pin="1"/>
+<pinref part="RESET" gate="S" pin="1"/>
 <wire x1="55.88" y1="48.26" x2="58.42" y2="48.26" width="0.1524" layer="91"/>
 <wire x1="58.42" y1="48.26" x2="58.42" y2="35.56" width="0.1524" layer="91"/>
-<pinref part="S1" gate="S" pin="2"/>
+<pinref part="RESET" gate="S" pin="2"/>
 <wire x1="58.42" y1="35.56" x2="58.42" y2="33.02" width="0.1524" layer="91"/>
 <pinref part="R1" gate="G$1" pin="1"/>
@@
 <pinref part="U1" gate="G$1" pin="SLEEVE"/>
 <pinref part="U1" gate="G$1" pin="RING"/>
-<wire x1="78.74" y1="99.06" x2="78.74" y2="96.52" width="0.1524" layer="91"/>
+<wire x1="78.74" y1="96.52" x2="78.74" y2="99.06" width="0.1524" layer="91"/>
 <pinref part="U1" gate="G$1" pin="RSH"/>
-<wire x1="78.74" y1="101.6" x2="78.74" y2="99.06" width="0.1524" layer="91"/>
+<wire x1="78.74" y1="99.06" x2="78.74" y2="101.6" width="0.1524" layer="91"/>
+<junction x="78.74" y="96.52"/>
 <junction x="78.74" y="99.06"/>
-<junction x="78.74" y="96.52"/>
 </segment>
 </net>
@@
 <segment>
 <pinref part="R4" gate="G$1" pin="2"/>
-<pinref part="LED1" gate="G$1" pin="A"/>
+<pinref part="STATUS" gate="G$1" pin="A"/>
 <wire x1="58.42" y1="73.66" x2="58.42" y2="76.2" width="0.1524" layer="91"/>
 </segment>

Commit message: Version 1.0 of the PCB
Gerber files for http://www.dorkbotpdx.org/wiki/pcb_order
Parts:
- added C3: 100nF, rcl:C-EU025-025X050
Connections:
- net +5V: now also C3.1
- net GND: now also C3.2
Changed lines of the file:
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@@
 <part name="U2" library="SparkFun" deviceset="AUDIO-JACK2" device="PTH" value="IR_Receiver"/>
 <part name="IC1" library="ATtiny85" deviceset="ATTINY85" device="DIP8"/>
+<part name="C3" library="rcl" deviceset="C-EU" device="025-025X050" value="100nF"/>
+<part name="GND8" library="supply1" deviceset="GND" device=""/>
 </parts>
 <sheets>
@@
 <instance part="GND1" gate="1" x="27.94" y="40.64"/>
 <instance part="GND3" gate="1" x="83.82" y="30.48"/>
-<instance part="P+1" gate="1" x="27.94" y="68.58"/>
+<instance part="P+1" gate="1" x="20.32" y="68.58"/>
 <instance part="RESET" gate="S" x="63.5" y="35.56"/>
 <instance part="R1" gate="G$1" x="50.8" y="33.02" rot="R180"/>
@@
 </instance>
 <instance part="IC1" gate="G$1" x="43.18" y="53.34"/>
+<instance part="C3" gate="G$1" x="20.32" y="55.88"/>
+<instance part="GND8" gate="1" x="20.32" y="45.72"/>
 </instances>
 <busses>
@@
 <wire x1="88.9" y1="63.5" x2="88.9" y2="60.96" width="0.1524" layer="91"/>
 </segment>
+<segment>
+<pinref part="C3" gate="G$1" pin="2"/>
+<pinref part="GND8" gate="1" pin="GND"/>
+<wire x1="20.32" y1="48.26" x2="20.32" y2="50.8" width="0.1524" layer="91"/>
+</segment>
 </net>
 <net name="N$1" class="0">
@@
 </net>
 <net name="+5V" class="0">
-<segment>
-<pinref part="P+1" gate="1" pin="+5V"/>
-<wire x1="27.94" y1="66.04" x2="27.94" y2="60.96" width="0.1524" layer="91"/>
-<pinref part="IC1" gate="G$1" pin="VCC"/>
-</segment>
 <segment>
 <pinref part="R1" gate="G$1" pin="2"/>
@@
 <junction x="88.9" y="73.66"/>
 </segment>
+<segment>
+<pinref part="P+1" gate="1" pin="+5V"/>
+<pinref part="C3" gate="G$1" pin="1"/>
+<wire x1="20.32" y1="58.42" x2="20.32" y2="60.96" width="0.1524" layer="91"/>
+<pinref part="IC1" gate="G$1" pin="VCC"/>
+<wire x1="20.32" y1="60.96" x2="20.32" y2="66.04" width="0.1524" layer="91"/>
+<wire x1="27.94" y1="60.96" x2="20.32" y2="60.96" width="0.1524" layer="91"/>
+<junction x="20.32" y="60.96"/>
+</segment>
 </net>
